Commit message: align boying config with go2: init joints, remove head collision, reduce terrain heights

File: resources/boying_description/urdf/boying_description.urdf (robot description, URDF)
Before this commit: robot boying, 20 links, 19 joints
Links:
- link head: geometry visual mesh filename=package://boying_description/meshes/head.STL

Commit message: 修复boying urdf，四条foot关节添加dont_collapse，统一足连杆命名

File: resources/boying_description/urdf/boying_description.urdf (robot description, URDF)
Before this commit: robot boying, 20 links, 19 joints
Links:
- removed link R_foot
- added link FR_foot, mass 0.052883; collision sphere radius=0.025; visual mesh filename=package://boying_description/meshes/R_foot.STL
- link FL_calf: geometry collision cylinder length=0.0564 radius=0.018; collision cylinder length=0.0647 radius=0.014000
- link FR_calf: geometry collision cylinder length=0.0564 radius=0.018; collision cylinder length=0.0647 radius=0.014000
- link RL_calf: geometry collision cylinder length=0.0564 radius=0.018; collision cylinder length=0.0647 radius=0.014000
- link RR_calf: geometry collision cylinder length=0.0564 radius=0.018; collision cylinder length=0.0647 radius=0.014000
Joints:
- removed joint R_foot_joint
- added joint FR_foot_joint: type fixed, parent FR_calf, child FR_foot, origin xyz=0 0 0 rpy=0 0 0, axis 0 0 0

Commit message: remove hm collision body; raise illegal_contact threshold 1->5N

File: resources/boying_description/urdf/boying_description.urdf (robot description, URDF)
Before this commit: robot boying, 20 links, 19 joints
Links:
- link hm: geometry visual mesh filename=package://boying_description/meshes/hm.STL

Commit message: fix FR/RR calf mass bug (0.051→0.138kg); split actuators, damping 4.5→2.0, calf vel_limit 10.4

File: resources/boying_description/urdf/boying_description.urdf (robot description, URDF)
Before this commit: robot boying, 20 links, 19 joints
Links:
- link FR_calf: mass 0.051104 -> 0.137980
- link RR_calf: mass 0.051104 -> 0.137980
